File: layout/C6MacroSwitch/layout.kicad_pcb (KiCad board)
At the start: 2 copper layers, 70 x 85 mm, 39 parts, among them J1 S2B-PH-K-S(LF)(SN), J2 61300211121, Q1 AO3401A, SW1 CPG135001D01, SW2 CPG135001D01, SW3 CPG135001D01, SW4 CPG135001D01, SW5 CPG135001D01, SW6 CPG135001D01, SW7 TSA061B2808B, SW8 TSA061B2808B, U1 ESP32-C6-WROOM-1-N8, U2 XC6220B331MR-G, U3 MCP73831T-2ACI/OT

Commit message: Kicad layout modded
Parts:
- moved USBC1 2.92 mm to (150.9, 129.7)
- moved R10 2.73 mm to (142.5, 128.1)
- moved R3 2.04 mm to (154.9, 123.5)
- moved SW8 1.51 mm to (141.8, 132.1)
- moved SW7 1.21 mm to (136.6, 132.0)
Routing:
- net GND: track 3.97 -> 29.7 mm, vias 8 -> 26
- net VBAT_SW: track 51.9 -> 49.0 mm
- net VBUS: track 35.5 -> 32.8 mm
- net CC2: track 6.60 -> 4.29 mm
- net 3V3: track 76.8 -> 79.1 mm
- net EN: track 17.6 -> 19.4 mm
- net VBAT_SENSE: track 11.5 -> 13.2 mm
- net CC1: track 7.40 -> 8.12 mm
- net USB_D_P: track 14.4 -> 13.7 mm
- net USB_D_N: track 13.8 -> 14.4 mm
Other:
- board text added: "Esp36C6 MacroButton 06/2026 V 1.0"
